Commit message: cuscobot TF review

File: urdf/lidar.xacro (robot description, xacro)
@@ -3,8 +3,8 @@
     <joint name="laser_joint" type="fixed">
         <parent link="chassis_link"/>
-        <child link="laser_frame"/>
+        <child link="laser"/>
         <origin xyz="0.125 0 0.2175" rpy="0 0 0"/>
     </joint>
-    <link name="laser_frame">
+    <link name="laser">
         <visual>
             <geometry>

File: urdf/robot.xacro (robot description, xacro)
@@ -38,4 +38,11 @@
 		<origin xyz= "0 0 0" />
 	</link>
+	<!-- base footprint -->>
+<!--	<joint name="base_footprint_joint">
+		<parent link ="base_joint"/>
+		<child link="base_footprint_joint"/>
+		<origin xyz="0 0 0" rpy="0 0 0"/>
+	</joint>
+-->
 	<!-- Chassis -->
 	<joint name="chassis_joint" type="fixed">

Commit message: nav_stacks tf working

File: urdf/lidar.xacro (robot description, xacro)
@@ -2,5 +2,5 @@
 <robot xmlns:xacro="http://www.ros.org/wiki/xacro" >
     <joint name="laser_joint" type="fixed">
-        <parent link="chassis_link"/>
+        <parent link="base_link"/>
         <child link="laser"/>
         <origin xyz="0.125 0 0.2175" rpy="0 0 0"/>

Commit message: amcl launch odom link

File: urdf/lidar.xacro (robot description, xacro)
@@ -4,5 +4,5 @@
         <parent link="base_link"/>
         <child link="laser"/>
-        <origin xyz="0.125 0 0.2175" rpy="0 0 0"/>
+        <origin xyz="0.04 0 0.305" rpy="0 0 0"/>
     </joint>
     <link name="laser">

File: urdf/robot.xacro (robot description, xacro)
@@ -38,11 +38,4 @@
 		<origin xyz= "0 0 0" />
 	</link>
-	<!-- base footprint -->>
-<!--	<joint name="base_footprint_joint">
-		<parent link ="base_joint"/>
-		<child link="base_footprint_joint"/>
-		<origin xyz="0 0 0" rpy="0 0 0"/>
-	</joint>
--->
 	<!-- Chassis -->
 	<joint name="chassis_joint" type="fixed">
